Commit message: working status deploying to robot

File: src/pcv_base/resources/cfg/omniveyor.urdf (robot description, URDF)
Before this commit: robot omniveyor, 5 links, 4 joints
Joints:
- joint laser_joint: origin xyz=0.27 0 0.1 rpy=0 0 0 -> xyz=0.27 0 0.15 rpy=0 0 0

Commit message: added configuration files for the robot to move in confined spaces (PVil tests). Fixed robot urdf definitions.

File: src/pcv_base/resources/cfg/omniveyor.urdf (robot description, URDF)
Before this commit: robot omniveyor, 5 links, 4 joints
Joints:
- joint rear_rs_joint: origin xyz=-0.4 0. 0.4 rpy=0. 0. 3.1416 -> xyz=-0.4 -0.08 0.4 rpy=0. 0. 3.1416

Commit message: Nov. testing batch update: door crossing, autorun code

File: src/pcv_base/resources/cfg/omniveyor.urdf (robot description, URDF)
Before this commit: robot omniveyor, 5 links, 4 joints
Joints:
- joint laser_joint: origin xyz=0.27 0 0.15 rpy=0 0 0 -> xyz=0.28 0 0.15 rpy=0 0 0
- joint rear_rs_joint: origin xyz=-0.4 -0.08 0.4 rpy=0. 0. 3.1416 -> xyz=-0.4 0. 0.4 rpy=0. 0. 3.1416

Commit message: added visual servoing with ArUco markers

File: src/pcv_base/resources/cfg/omniveyor.urdf (robot description, URDF)
Before this commit: robot omniveyor, 5 links, 4 joints
Joints:
- joint front_rs_joint: origin xyz=0.4 0.08 0.4 rpy=0. 0. 0. -> xyz=0.285 0.08 0.4 rpy=0. 0. 0.
- joint front_t265_joint: origin xyz=0.4 -0.08 0.4 rpy=0. 0. 0. -> xyz=0.285 -0.08 0.4 rpy=0. 0. 0.
- joint laser_joint: origin xyz=0.28 0 0.15 rpy=0 0 0 -> xyz=0.28 0 0.11 rpy=0 0 0
- joint rear_rs_joint: origin xyz=-0.4 0. 0.4 rpy=0. 0. 3.1416 -> xyz=-0.285 -0.08 0.4 rpy=0. 0. 3.1416
